File: pcb/mikeneko-65-pcb.kicad_pcb (KiCad board)
At the start: 2 copper layers, 303.8 x 94.2 mm, 161 parts, among them J1 JST SH 4-pin, J2 AVR-ISP-6, SW1 Reset, U1 SRV05-4, U2 ATmega32U4-AU, Y1 16MHz

Commit message: bakenekoをmikenekoに変換。
Parts:
- J2: footprint bakeneko:ISP -> mikeneko:ISP
Other:
- board text added: "Mikeneko65 v3.0"
- board text removed: "Bakeneko65 v3.0"
Changed lines of the file:
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@@
     (add_net VBUS)
   )
-  (module bakeneko:ISP (layer B.Cu)
+  (module mikeneko:ISP (layer B.Cu)
     (at 5.19 20.807501)
     (descr "6-pin AVR ISP")
@@
   (gr_arc (start 262.051894 92.7) (end 262.051894 94.2) (angle -62.46013955) (layer Edge.Cuts) (width 0.2))
   (gr_arc (start 266.175 94.85) (end 268.968071 93.393549) (angle -124.9202791) (layer Edge.Cuts) (width 0.2))
-  (gr_text "Bakeneko65 v3.0" (at 293.965477 91.907501) (layer B.SilkS)
+  (gr_text "Mikeneko65 v3.0" (at 293.965477 91.907501) (layer B.SilkS)
     (effects (font (size 1 1) (thickness 0.15)) (justify mirror))
   )
