File: pcb/mikeneko-65-pcb.kicad_pcb (KiCad board)
At the start: 2 copper layers, 303.8 x 94.2 mm, 161 parts, among them J1 JST SH 4-pin, J2 AVR-ISP-6, SW1 Reset, U1 SRV05-4, U2 ATmega32U4-MU, Y1 16MHz

Commit message: ソケットに対応。
Parts:
- removed the D14 at (247.1, 9.79)
- removed the MX14 at (256.6, 9.00)
- removed the MX15 at (275.7, 9.00)
- removed the MX33 at (11.4, 47.1)
- removed the MX62 at (13.8, 85.2)
- removed the MX63 at (37.6, 85.2)
- removed the MX64 at (61.4, 85.2)
- removed the MX65 at (142.3, 85.2)
- removed the MX67 at (223.3, 85.2)
- J2: moved to F.Cu
- MX1, MX10, MX11, MX12, MX13, MX2, MX3, MX4, MX5, MX6, MX7, MX8, MX9: footprint MX_Only:MXOnly-1U-NoLED -> MX_Only:MXOnly-1U-Hotswap
- MX14: renamed from MX17; footprint MX_Only:MXOnly-2U-NoLED -> MX_Only:MXOnly-2U-Hotswap
- MX15: renamed from MX16; footprint MX_Only:MXOnly-1U-NoLED -> MX_Only:MXOnly-1U-Hotswap
- MX16: renamed from MX18; footprint MX_Only:MXOnly-1.5U-NoLED -> MX_Only:MXOnly-1.5U-Hotswap
- MX17: renamed from MX19; footprint MX_Only:MXOnly-1U-NoLED -> MX_Only:MXOnly-1U-Hotswap
- MX18: renamed from MX20; footprint MX_Only:MXOnly-1U-NoLED -> MX_Only:MXOnly-1U-Hotswap
- MX19: renamed from MX21; footprint MX_Only:MXOnly-1U-NoLED -> MX_Only:MXOnly-1U-Hotswap
- MX20: renamed from MX22; footprint MX_Only:MXOnly-1U-NoLED -> MX_Only:MXOnly-1U-Hotswap
- MX21: renamed from MX23; footprint MX_Only:MXOnly-1U-NoLED -> MX_Only:MXOnly-1U-Hotswap
- MX22: renamed from MX24; footprint MX_Only:MXOnly-1U-NoLED -> MX_Only:MXOnly-1U-Hotswap
- MX23: renamed from MX25; footprint MX_Only:MXOnly-1U-NoLED -> MX_Only:MXOnly-1U-Hotswap
- MX24: renamed from MX26; footprint MX_Only:MXOnly-1U-NoLED -> MX_Only:MXOnly-1U-Hotswap
- MX25: renamed from MX27; footprint MX_Only:MXOnly-1U-NoLED -> MX_Only:MXOnly-1U-Hotswap
- MX26: renamed from MX28; footprint MX_Only:MXOnly-1U-NoLED -> MX_Only:MXOnly-1U-Hotswap
- MX27: renamed from MX29; footprint MX_Only:MXOnly-1U-NoLED -> MX_Only:MXOnly-1U-Hotswap
- MX28: renamed from MX30; footprint MX_Only:MXOnly-1U-NoLED -> MX_Only:MXOnly-1U-Hotswap
- MX29: renamed from MX31; footprint MX_Only:MXOnly-1.5U-NoLED -> MX_Only:MXOnly-1.5U-Hotswap
- MX30: renamed from MX32; footprint MX_Only:MXOnly-1U-NoLED -> MX_Only:MXOnly-1U-Hotswap
- MX31: renamed from MX34; footprint MX_Only:MXOnly-1.75U-NoLED -> MX_Only:MXOnly-1.75U-Hotswap
- MX32: renamed from MX35; footprint MX_Only:MXOnly-1U-NoLED -> MX_Only:MXOnly-1U-Hotswap
- MX33: renamed from MX36; footprint MX_Only:MXOnly-1U-NoLED -> MX_Only:MXOnly-1U-Hotswap
- MX34: renamed from MX37; footprint MX_Only:MXOnly-1U-NoLED -> MX_Only:MXOnly-1U-Hotswap
- MX35: renamed from MX38; footprint MX_Only:MXOnly-1U-NoLED -> MX_Only:MXOnly-1U-Hotswap
- MX36: renamed from MX39; footprint MX_Only:MXOnly-1U-NoLED -> MX_Only:MXOnly-1U-Hotswap
- MX37: renamed from MX40; footprint MX_Only:MXOnly-1U-NoLED -> MX_Only:MXOnly-1U-Hotswap
- MX38: renamed from MX41; footprint MX_Only:MXOnly-1U-NoLED -> MX_Only:MXOnly-1U-Hotswap
- MX39: renamed from MX42; footprint MX_Only:MXOnly-1U-NoLED -> MX_Only:MXOnly-1U-Hotswap
- MX40: renamed from MX43; footprint MX_Only:MXOnly-1U-NoLED -> MX_Only:MXOnly-1U-Hotswap
- MX41: renamed from MX44; footprint MX_Only:MXOnly-1U-NoLED -> MX_Only:MXOnly-1U-Hotswap
- MX42: renamed from MX45; footprint MX_Only:MXOnly-1U-NoLED -> MX_Only:MXOnly-1U-Hotswap
- MX43: renamed from MX46; footprint MX_Only:MXOnly-2.25U-NoLED -> MX_Only:MXOnly-2.25U-Hotswap
- MX44: renamed from MX47; footprint MX_Only:MXOnly-1U-NoLED -> MX_Only:MXOnly-1U-Hotswap
- MX45: renamed from MX48; footprint MX_Only:MXOnly-2.25U-NoLED -> MX_Only:MXOnly-2.25U-Hotswap
- MX46: renamed from MX49; footprint MX_Only:MXOnly-1U-NoLED -> MX_Only:MXOnly-1U-Hotswap
- MX47: renamed from MX50; footprint MX_Only:MXOnly-1U-NoLED -> MX_Only:MXOnly-1U-Hotswap
- MX48: renamed from MX51; footprint MX_Only:MXOnly-1U-NoLED -> MX_Only:MXOnly-1U-Hotswap
- MX49: renamed from MX52; footprint MX_Only:MXOnly-1U-NoLED -> MX_Only:MXOnly-1U-Hotswap
- MX50: renamed from MX53; footprint MX_Only:MXOnly-1U-NoLED -> MX_Only:MXOnly-1U-Hotswap
- MX51: renamed from MX54; footprint MX_Only:MXOnly-1U-NoLED -> MX_Only:MXOnly-1U-Hotswap
- MX52: renamed from MX55; footprint MX_Only:MXOnly-1U-NoLED -> MX_Only:MXOnly-1U-Hotswap
- MX53: renamed from MX56; footprint MX_Only:MXOnly-1U-NoLED -> MX_Only:MXOnly-1U-Hotswap
- MX54: renamed from MX57; footprint MX_Only:MXOnly-1U-NoLED -> MX_Only:MXOnly-1U-Hotswap
- MX55: renamed from MX58; footprint MX_Only:MXOnly-1U-NoLED -> MX_Only:MXOnly-1U-Hotswap
- MX56: renamed from MX59; footprint MX_Only:MXOnly-1.75U-NoLED -> MX_Only:MXOnly-1.75U-Hotswap
- MX57: renamed from MX60; footprint MX_Only:MXOnly-1U-NoLED -> MX_Only:MXOnly-1U-Hotswap
- MX58: renamed from MX61; footprint MX_Only:MXOnly-1U-NoLED -> MX_Only:MXOnly-1U-Hotswap
- MX59: renamed from MX71; footprint MX_Only:MXOnly-1.25U-NoLED -> MX_Only:MXOnly-1.25U-Hotswap
- MX60: renamed from MX72; footprint MX_Only:MXOnly-1.25U-NoLED -> MX_Only:MXOnly-1.25U-Hotswap
- MX61: renamed from MX73; footprint MX_Only:MXOnly-1.25U-NoLED -> MX_Only:MXOnly-1.25U-Hotswap
- MX62: renamed from MX74; footprint MX_Only:MXOnly-6.25U-ReversedStabilizers-NoLED -> MX_Only:MXOnly-6.25U-Hotswap-ReversedStabilizers
- MX63: renamed from MX66; footprint MX_Only:MXOnly-1.25U-NoLED -> MX_Only:MXOnly-1.25U-Hotswap
- MX64: renamed from MX75; footprint MX_Only:MXOnly-1.25U-NoLED -> MX_Only:MXOnly-1.25U-Hotswap
- MX65: renamed from MX68; footprint MX_Only:MXOnly-1U-NoLED -> MX_Only:MXOnly-1U-Hotswap
- MX66: renamed from MX69; footprint MX_Only:MXOnly-1U-NoLED -> MX_Only:MXOnly-1U-Hotswap
- MX67: renamed from MX70; footprint MX_Only:MXOnly-1U-NoLED -> MX_Only:MXOnly-1U-Hotswap
- moved J2 168.9 mm to (165.9, 72.8), turned to 270 degrees
- moved C3 134.8 mm to (160.0, 89.5), turned to 180 degrees
- moved C1 134.5 mm to (162.7, 82.0)
- moved C2 134.5 mm to (142.7, 86.7)
- moved C4 134.5 mm to (148.7, 76.9)
- moved C5 134.5 mm to (166.5, 83.0)
- moved C6 134.5 mm to (166.5, 88.6)
- moved C7 134.5 mm to (153.7, 75.6)
- moved R1 134.5 mm to (175.3, 82.7)
- moved SW1 134.5 mm to (180.8, 83.6)
- moved U2 134.5 mm to (154.1, 85.8)
- moved Y1 134.5 mm to (166.5, 85.8)
- moved R4 117.9 mm to (142.9, 89.1), turned to 0 degrees
- moved D17 39.2 mm to (28.6, 31.0)
- moved D14 26.5 mm to (257.2, 11.9)
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- renumbered D15 to D14, D16 to D15, D17 to D16, D18 to D17, D19 to D18, D20 to D19, D21 to D20, D22 to D21, D23 to D22, D24 to D23, D25 to D24, D26 to D25, D27 to D26, D28 to D27, D29 to D28, D30 to D29, D31 to D30, D32 to D31, D33 to D32, D34 to D33, D35 to D34, D36 to D35, D37 to D36, D38 to D37, D39 to D38, D40 to D39, D41 to D40, D42 to D41, D43 to D42, D44 to D43, D45 to D44, D46 to D45, D47 to D46, D48 to D47, D49 to D48, D50 to D49, D51 to D50, D52 to D51, D53 to D52, D54 to D53, D55 to D54, D56 to D55, D57 to D56, D58 to D57, D59 to D58, D60 to D59, D61 to D60, D62 to D61, D63 to D62, D64 to D63, D65 to D64, D66 to D65, D67 to D66, D68 to D67
Connections:
- MX14 pad 2: COL14 -> COL13
- MX15 pad 2: COL15 -> COL14
- MX30 pad 2: COL15 -> COL14
- MX44 pad 2: COL15 -> COL14
- MX58 pad 2: COL15 -> COL14
- MX67 pad 2: COL15 -> COL14
- U2 pad 1: ROW0 -> COL6
- U2 pad 12: ROW1 -> COL8
- U2 pad 18: COL15 -> COL9
- U2 pad 19: COL14 -> COL10
- U2 pad 20: COL13 -> COL11
- U2 pad 22: COL11 -> COL13
- U2 pad 25: COL10 -> COL14
- U2 pad 26: COL9 -> ROW1
- U2 pad 27: COL8 -> ROW0
- U2 pad 28: COL7 -> Net-(U2-Pad28)
- U2 pad 29: COL6 -> Net-(U2-Pad29)
- U2 pad 30: COL5 -> ROW2
- U2 pad 31: COL4 -> ROW3
- U2 pad 32: COL3 -> ROW4
- U2 pad 36: ROW2 -> COL0
- U2 pad 37: COL0 -> COL1
- U2 pad 38: ROW4 -> COL2
- U2 pad 39: ROW3 -> COL3
- U2 pad 40: COL2 -> COL4
- U2 pad 41: Net-(U2-Pad41) -> COL5
- U2 pad 8: COL1 -> COL7
Routing:
- net COL15: track 356.4 -> 0.00 mm
- net ROW0: track 298.2 -> 551.0 mm, vias 2 -> 3
- net +5V: track 139.1 -> 326.1 mm, vias 6 -> 7
- net GND: track 185.2 -> 357.4 mm, vias 5 -> 3
- net /MCU_D-: track 21.9 -> 193.4 mm, vias 0 -> 4
- net /MCU_D+: track 20.9 -> 191.5 mm, vias 0 -> 4
- net COL13: track 354.7 -> 227.5 mm, vias 0 -> 9
- net COL11: track 295.4 -> 169.9 mm, vias 0 -> 10
- net COL0: track 102.4 -> 227.4 mm, vias 1 -> 11
- net COL9: track 268.5 -> 147.4 mm, vias 0 -> 9
- net COL12: track 320.1 -> 200.4 mm, vias 0 -> 7
- net COL8: track 219.4 -> 99.7 mm, vias 0 -> 8
- net COL10: track 256.4 -> 137.8 mm, vias 0 -> 8
- net COL7: track 200.9 -> 92.3 mm, vias 0 -> 8
- net COL6: track 214.6 -> 109.6 mm, vias 0 -> 10
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
Commit message: 配線を更新。
Parts:
- moved MX66 0.05 mm to (275.8, 85.2)
Connections:
- U2 pad 18: COL9 -> ROW0
- U2 pad 19: COL10 -> Net-(U2-Pad19)
- U2 pad 20: COL11 -> ROW1
- U2 pad 21: COL12 -> Net-(U2-Pad21)
- U2 pad 22: COL13 -> ROW2
- U2 pad 25: COL14 -> COL9
- U2 pad 26: ROW1 -> COL10
- U2 pad 27: ROW0 -> COL11
- U2 pad 28: Net-(U2-Pad28) -> COL14
- U2 pad 29: Net-(U2-Pad29) -> COL13
- U2 pad 30: ROW2 -> COL12
Routing:
- net ROW0: track 551.0 -> 372.3 mm, vias 3 -> 2
- net COL1: track 203.3 -> 246.7 mm, vias 6 -> 8
- net +5V: track 326.1 -> 285.1 mm
- net ROW2: track 375.8 -> 337.8 mm, vias 2 -> 4
- net GND: track 357.4 -> 324.4 mm
- net COL3: track 199.0 -> 172.8 mm
- net ROW1: track 374.1 -> 354.0 mm, vias 2 -> 4
- net COL10: track 137.8 -> 153.1 mm
- net COL12: track 200.4 -> 213.9 mm, vias 7 -> 8
- net COL4: track 140.3 -> 151.8 mm
- net COL13: track 227.5 -> 234.9 mm, vias 9 -> 8
- net ROW4: track 324.0 -> 317.5 mm
- net COL9: track 147.4 -> 153.7 mm, vias 9 -> 8
- net COL11: track 169.9 -> 175.4 mm, vias 10 -> 9
- net COL5: track 122.2 -> 127.1 mm
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
Commit message: V3をV4に変更。
Other:
- board text added: "Mikeneko65 v4.0"
- board text removed: "Mikeneko65 v3.0"
Changed lines of the file:
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@@
   (gr_arc (start 262.051894 92.7) (end 262.051894 94.2) (angle -62.46013955) (layer Edge.Cuts) (width 0.2))
   (gr_arc (start 266.175 94.85) (end 268.968071 93.393549) (angle -124.9202791) (layer Edge.Cuts) (width 0.2))
-  (gr_text "Mikeneko65 v3.0" (at 293.965477 91.907501) (layer B.SilkS)
+  (gr_text "Mikeneko65 v4.0" (at 293.965477 91.907501) (layer B.SilkS)
     (effects (font (size 1 1) (thickness 0.15)) (justify mirror))
   )
