File: pcb/mikeneko-65-pcb.sch (KiCad schematic (older format))
At the start: 18 parts, among them J1 JST SH 4-pin, J2 AVR-ISP-6, SW1 Reset, U1 SRV05-4, U2 ATmega32U4-AU, Y1 16MHz

Commit message: bakenekoをmikenekoに変換。
Parts:
- J2: footprint bakeneko:ISP -> mikeneko:ISP
Changed lines of the file:
@@
 EESchema Schematic File Version 4
-LIBS:bakeneko-65-pcb-cache
+LIBS:mikeneko-65-pcb-cache
 EELAYER 30 0
 EELAYER END
@@
 encoding utf-8
 Sheet 1 2
-Title "Bakeneko 65 V3"
+Title "Mikeneko 65 V3"
 Date "2020-08-01"
 Rev "1"
@@
 F 0 "J2" H 1721 1796 50  0000 R CNN
 F 1 "AVR-ISP-6" H 1721 1705 50  0000 R CNN
-F 2 "bakeneko:ISP" V 1800 1750 50  0001 C CNN
+F 2 "mikeneko:ISP" V 1800 1750 50  0001 C CNN
 F 3 " ~" H 775 1150 50  0001 C CNN
 	1    2050 1700
