File: plate/fr4/mikeneko-65-fr4-plate.kicad_pcb (KiCad board)
At the start: 2 copper layers, 304.8 x 95.2 mm, 0 parts

Commit message: スクリューインタイプのスタビライザーに対応し、ガーバーファイルを更新。
Other:
- board size 304.8 x 95.2 mm -> 304.8 x 95.3 mm
